File: sch_pcb/adc_40MHz/adc_40MHz.sch (EAGLE design)
At the start: 0 parts

Commit message: Dodano drabinki rezystorowe do biblioteki. Rozpoczęto prace nad schematem
Parts:
- added C1, C5, C6: 100n, rcl:C-EUC0603
- added C2: (no value), rcl:C-EUC0603
- added C3, C4: (no value), rcl:C-EUC0805
- added C7: 51p, rcl:C-EUC0603
- added IC1: (no value), lt6600:LT6600-15
- added IC2: AD9235BC, ad9235:AD9235BC
- added IC3, IC4: (no value), ltc625x:LTC6252
- added R1, R2, R5: (no value), rcl:R-EU_R0603
- added R3, R4: 40, rcl:R-EU_R0603
- added RN1, RN2, RN3: 100, passive:CTS742C083
- added SV1: (no value), con-harting-ml:ML26
- added X1, X2: BU-SMA-H, con-coax:BU-SMA-H
Connections:
- new net ADC_D0: IC2.D0, RN3.4
- new net ADC_D1: IC2.D1, RN3.3
- new net ADC_D10: IC2.D10, RN1.2
- new net ADC_D11: IC2.D11, RN1.1
- new net ADC_D2: IC2.D2, RN3.2
- new net ADC_D3: IC2.D3, RN3.1
- new net ADC_D4: IC2.D4, RN2.4
- new net ADC_D5: IC2.D5, RN2.3
- new net ADC_D6: IC2.D6, RN2.2
- new net ADC_D7: IC2.D7, RN2.1
- new net ADC_D8: IC2.D8, RN1.4
- new net ADC_D9: IC2.D9, RN1.3
- new net DAC_D0: RN3.5, SV1.23
- new net DAC_D1: RN3.6, SV1.21
- new net DAC_D10: RN1.7, SV1.3
- new net DAC_D11: RN1.8, SV1.1
- new net DAC_D2: RN3.7, SV1.19
- new net DAC_D3: RN3.8, SV1.17
- new net DAC_D4: RN2.5, SV1.15
- new net DAC_D5: RN2.6, SV1.13
- new net DAC_D6: RN2.7, SV1.11
- new net DAC_D7: RN2.8, SV1.9
- new net DAC_D8: RN1.5, SV1.7
- new net DAC_D9: RN1.6, SV1.5
- new net GND: IC2.AGND, IC2.DGND, SV1.10, SV1.12, SV1.14, SV1.16, SV1.18, SV1.2, SV1.20, SV1.22, SV1.24, SV1.26, SV1.4, SV1.6, SV1.8, X1.2, X2.2
- new net N$1: IC1.OUT+, R3.1
- new net N$2: C7.1, IC2.VIN+, R3.2
- new net N$3: C7.2, IC2.VIN-, R4.2
- new net N$4: IC1.OUT-, R4.1
- new net N$7: IC2.CLK, SV1.25, X2.1
