File: sch_pcb/adc_40MHz/adc_40MHz_v3.brd (EAGLE design)
At the start: 99 x 54.3 mm, 63 parts, among them IC1 LTC2227, IC2 LT6600-15, IC3 LTC6254XMS, IC5 LT1521XST, X1 SIGNAL, X2 CLK

Commit message: pboard
pboard
Routing:
- net +3V3: track 214.3 -> 235.7 mm, vias 9 -> 10
- net N$20: track 3.81 -> 13.5 mm, vias 0 -> 2
- net GND: track 58.6 -> 64.5 mm
Changed lines of the file:
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@@
 <wire x1="67.465" y1="61.75" x2="68.72" y2="61.75" width="0.254" layer="1"/>
 <wire x1="67.465" y1="58.9" x2="67.465" y2="61.75" width="0.254" layer="1"/>
-<wire x1="73.52" y1="63.25" x2="71.12" y2="63.5" width="0" layer="19" extent="1-1"/>
-<wire x1="52.49" y1="80.01" x2="49.911" y2="77.724" width="0" layer="19" extent="1-1"/>
+<wire x1="72.9488" y1="63.3984" x2="71.12" y2="63.3984" width="0.2032" layer="1"/>
+<wire x1="73.152" y1="63.1952" x2="72.9488" y2="63.3984" width="0.2032" layer="1"/>
+<wire x1="73.3552" y1="63.1952" x2="73.152" y2="63.1952" width="0.2032" layer="1"/>
+<wire x1="73.3552" y1="63.1952" x2="73.52" y2="63.25" width="0.2032" layer="1"/>
+<wire x1="69.4944" y1="61.7728" x2="71.12" y2="63.3984" width="0.2032" layer="1"/>
+<wire x1="69.088" y1="61.7728" x2="69.4944" y2="61.7728" width="0.2032" layer="1"/>
+<wire x1="68.6816" y1="61.3664" x2="69.088" y2="61.7728" width="0.2032" layer="1"/>
+<wire x1="71.12" y1="63.3984" x2="71.12" y2="63.5" width="0.2032" layer="1"/>
+<wire x1="68.6816" y1="61.3664" x2="68.6816" y2="61.294796875" width="0.2032" layer="1"/>
+<wire x1="49.911" y1="77.724" x2="52.49" y2="80.01" width="0" layer="19" extent="1-1"/>
 <wire x1="48.895" y1="54.014" x2="53.66" y2="54.61" width="0" layer="19" extent="1-1"/>
 <wire x1="52.07" y1="64.35" x2="50.8" y2="70.8" width="0" layer="19" extent="1-1"/>
@@
 <wire x1="61.81" y1="43.18" x2="61.81" y2="46.99" width="0.254" layer="1"/>
 <wire x1="61.81" y1="46.99" x2="61.81" y2="50.8" width="0.254" layer="1"/>
-<wire x1="55.56" y1="46.99" x2="55.56" y2="43.18" width="0.254" layer="1"/>
+<wire x1="55.56" y1="46.99" x2="55.56" y2="45.1104" width="0.254" layer="1"/>
+<wire x1="55.56" y1="45.1104" x2="55.56" y2="43.18" width="0.254" layer="1"/>
 <wire x1="55.56" y1="54.61" x2="63.5" y2="54.61" width="0.254" layer="1"/>
 <wire x1="63.5" y1="54.61" x2="63.5" y2="50.8" width="0.254" layer="1"/>
@@
 <wire x1="69.37" y1="66.774" x2="69.37" y2="65.9" width="0.254" layer="1"/>
 <wire x1="64.77" y1="54.61" x2="65.024" y2="54.864" width="0.254" layer="16"/>
-<wire x1="65.024" y1="54.864" x2="65.024" y2="66.675" width="0.254" layer="16"/>
+<wire x1="65.024" y1="54.864" x2="65.024" y2="58.7248" width="0.254" layer="16"/>
 <via x="65.024" y="66.675" extent="1-16" drill="0.508"/>
+<wire x1="65.024" y1="58.7248" x2="65.024" y2="66.675" width="0.254" layer="16"/>
 <wire x1="65.024" y1="66.675" x2="65.024" y2="67.31" width="0.254" layer="1"/>
 <wire x1="53.34" y1="67.31" x2="60.96" y2="67.31" width="0.254" layer="1"/>
@@
 <wire x1="76.454" y1="64.135" x2="76.073" y2="63.754" width="0.254" layer="1"/>
 <wire x1="76.073" y1="63.754" x2="73.524" y2="63.754" width="0.254" layer="1"/>
-<wire x1="61.81" y1="43.18" x2="55.56" y2="43.18" width="0" layer="19" extent="1-1"/>
+<wire x1="55.4736" y1="45.1104" x2="55.6768" y2="45.1104" width="0.2032" layer="16"/>
+<wire x1="55.4736" y1="55.0672" x2="55.4736" y2="45.1104" width="0.2032" layer="16"/>
+<wire x1="59.1312" y1="58.7248" x2="55.4736" y2="55.0672" width="0.2032" layer="16"/>
+<wire x1="65.024" y1="58.7248" x2="59.1312" y2="58.7248" width="0.2032" layer="16"/>
+<wire x1="55.6768" y1="45.1104" x2="55.56" y2="45.1104" width="0.2032" layer="1"/>
+<via x="55.6768" y="45.1104" extent="1-16" drill="0.3"/>
 </signal>
 <signal name="N$6">
@@
 <contactref element="R20" pad="1"/>
 <contactref element="R17" pad="1"/>
-<wire x1="14.39" y1="74.93" x2="14.39" y2="71.12" width="0.254" layer="1"/>
-<wire x1="14.39" y1="74.93" x2="14.39" y2="78.74" width="0" layer="19" extent="1-1"/>
-<wire x1="14.39" y1="67.31" x2="14.39" y2="71.12" width="0" layer="19" extent="1-1"/>
+<wire x1="14.39" y1="74.93" x2="14.39" y2="73.7616" width="0.254" layer="1"/>
+<wire x1="14.39" y1="73.7616" x2="14.39" y2="71.12" width="0.254" layer="1"/>
+<wire x1="14.4272" y1="71.12" x2="14.4272" y2="67.4624" width="0.2032" layer="1"/>
+<wire x1="14.4272" y1="67.4624" x2="14.39" y2="67.31" width="0.2032" layer="1"/>
+<wire x1="14.4272" y1="71.12" x2="14.39" y2="71.12" width="0.2032" layer="1"/>
+<wire x1="13.4112" y1="77.8256" x2="14.224" y2="78.6384" width="0.2032" layer="1"/>
+<wire x1="13.4112" y1="74.7776" x2="13.4112" y2="77.8256" width="0.2032" layer="16"/>
+<wire x1="14.4272" y1="73.7616" x2="13.4112" y2="74.7776" width="0.2032" layer="16"/>
+<wire x1="14.224" y1="78.6384" x2="14.39" y2="78.74" width="0.2032" layer="1"/>
+<wire x1="14.4272" y1="73.7616" x2="14.39" y2="73.7616" width="0.2032" layer="1"/>
+<via x="13.4112" y="77.8256" extent="1-16" drill="0.3"/>
+<via x="14.4272" y="73.7616" extent="1-16" drill="0.3"/>
 </signal>
 <signal name="N$21">
