File: sch_pcb/adc_40MHz/adc_40MHz.brd (EAGLE design)
At the start: 66 x 40.6 mm, 74 parts, among them IC1 AD9235BC, IC2 LT6600-15, IC3 LTC6254XMS, IC4 SN74LVC2G14DBV, IC5 LT1521XST, IC6 SN74LVC2G14DBV, X1 SMA-142-0701-851/861, X2 SMA-142-0701-851/861

Commit message: Dodano BOM, poprawiono wartości niektórych rezystancji
Parts:
- R1: value 430 -> 430R
- R3, R4: value 40 -> 40R
Changed lines of the file:
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@@
 <element name="C5" library="resistor" package="C0603K" value="100n" x="25.146" y="28.194" rot="R90"/>
 <element name="C7" library="resistor" package="C0603K" value="51p" x="35.814" y="21.844" rot="R90"/>
-<element name="R3" library="rcl" package="R0603" value="40" x="33.528" y="24.384"/>
-<element name="R4" library="rcl" package="R0603" value="40" x="33.528" y="22.86"/>
+<element name="R3" library="rcl" package="R0603" value="40R" x="33.528" y="24.384"/>
+<element name="R4" library="rcl" package="R0603" value="40R" x="33.528" y="22.86"/>
 <element name="R5" library="rcl" package="R0603" value="2.4k" x="17.018" y="34.036"/>
 <element name="RN1" library="passive" package="EXB38V" value="100R" x="53.34" y="28.448" rot="R270"/>
@@
 <element name="R11" library="rcl" package="R0603" value="20k" x="49.276" y="32.258" rot="R270"/>
 <element name="R12" library="rcl" package="R0603" value="10k" x="47.879" y="32.258" rot="R270"/>
-<element name="R1" library="rcl" package="R0603" value="430" x="17.018" y="32.512" rot="R180"/>
+<element name="R1" library="rcl" package="R0603" value="430R" x="17.018" y="32.512" rot="R180"/>
 <element name="C1" library="resistor" package="C0603K" value="20p" x="20.32" y="32.512" rot="R180"/>
 <element name="C2" library="resistor" package="C0603K" value="5p" x="17.018" y="30.988"/>
